Commit message: clean up initial code

File: data/a1/a1_urdf/a1.urdf (robot description, URDF)
Before this commit: robot a1_description, 23 links, 22 joints
Links:
- link FL_calf: geometry collision box size=0.2 0.016 0.016; visual mesh filename=.//calf.STL scale=1 1 1
- link FL_hip: geometry collision cylinder length=0.04 radius=0.046; visual mesh filename=.//hip.STL scale=1 1 1
- link FL_thigh: geometry collision box size=0.2 0.0245 0.034; visual mesh filename=.//thigh.STL scale=1 1 1
- link FR_calf: geometry collision box size=0.2 0.016 0.016; visual mesh filename=.//calf.STL scale=1 1 1
- link FR_hip: geometry collision cylinder length=0.04 radius=0.046; visual mesh filename=.//hip.STL scale=1 1 1
- link FR_thigh: geometry collision box size=0.2 0.0245 0.034; visual mesh filename=.//thigh_mirror.STL scale=1 1 1
- link RL_calf: geometry collision box size=0.2 0.016 0.016; visual mesh filename=.//calf.STL scale=1 1 1
- link RL_hip: geometry collision cylinder length=0.04 radius=0.046; visual mesh filename=.//hip.STL scale=1 1 1
- link RL_thigh: geometry collision box size=0.2 0.0245 0.034; visual mesh filename=.//thigh.STL scale=1 1 1
- link RR_calf: geometry collision box size=0.2 0.016 0.016; visual mesh filename=.//calf.STL scale=1 1 1
- link RR_hip: geometry collision cylinder length=0.04 radius=0.046; visual mesh filename=.//hip.STL scale=1 1 1
- link RR_thigh: geometry collision box size=0.2 0.0245 0.034; visual mesh filename=.//thigh_mirror.STL scale=1 1 1
- link trunk: geometry collision box size=0.267 0.194 0.114; visual mesh filename=.//trunk.STL scale=1 1 1

File: data/a1/a1_urdf/leg.xacro (robot description, xacro)
@@ -31,5 +31,5 @@
                 </xacro:if>
                 <geometry>
-                    <mesh filename="package://data/A1/meshes/hip.stl" scale="1 1 1"/>
+                    <mesh filename=".//hip.stl" scale="1 1 1"/>
                 </geometry>
                 <material name="orange"/>
@@ -77,8 +77,8 @@
                 <geometry>
                     <xacro:if value="${mirror_dae == True}">
-                        <mesh filename="package://data/A1/meshes/thigh.stl" scale="1 1 1"/>
+                        <mesh filename=".//thigh.stl" scale="1 1 1"/>
                     </xacro:if>
                     <xacro:if value="${mirror_dae == False}">
-                        <mesh filename="package://data/A1/meshes/thigh_mirror.stl" scale="1 1 1"/>
+                        <mesh filename=".//thigh_mirror.stl" scale="1 1 1"/>
                     </xacro:if>
                 </geometry>
@@ -112,5 +112,5 @@
                 <origin rpy="0 0 0" xyz="0 0 0"/>
                 <geometry>
-                    <mesh filename="package://data/A1/meshes/calf.stl" scale="1 1 1"/>
+                    <mesh filename=".//calf.stl" scale="1 1 1"/>
                 </geometry>
                 <material name="orange"/>

File: data/a1/a1_urdf/robot.xacro (robot description, xacro)
@@ -36,5 +36,5 @@
             <origin rpy="0 0 0" xyz="0 0 0"/>
             <geometry>
-                <mesh filename="package://data/A1/meshes/trunk.stl" scale="1 1 1"/>
+                <mesh filename=".//trunk.stl" scale="1 1 1"/>
             </geometry>
             <material name="orange"/>
