Commit message: create env

File: unitree_env/unitree_data/a1/a1_urdf/a1_eva_01.urdf (robot description, URDF)
Before this commit: robot a1_description, 23 links, 22 joints
Links:
- link FL_thigh_shoulder: geometry collision cylinder length=0.032 radius=0.041; visual mesh filename=.//hip.STL scale=1 1 1
- link FR_thigh_shoulder: geometry collision cylinder length=0.032 radius=0.041; visual mesh filename=.//hip.STL scale=1 1 1
- link RL_thigh_shoulder: geometry collision cylinder length=0.032 radius=0.041; visual mesh filename=.//hip.STL scale=1 1 1
- link RR_thigh_shoulder: geometry collision cylinder length=0.032 radius=0.041; visual mesh filename=.//hip.STL scale=1 1 1

File: unitree_env/unitree_data/a1/a1_urdf/materials.xacro (robot description, xacro)
@@ -25,5 +25,5 @@
         <color rgba="0.8 0.0 0.0 1.0"/>
     </material>
-    <material name="white">
+    <material name="grey">
         <color rgba="1.0 1.0 1.0 1.0"/>
     </material>
